Commit message: improved link positions and inertia

File: dronesim/assets/Falcon_opt.urdf (robot description, URDF)
Before this commit: robot Falcon, 6 links, 5 joints
Links:
- added link aerodynamic_center_link, mass 0
Joints:
- added joint aerodynamic_center_joint: type fixed, parent base_link, child aerodynamic_center_link
